Commit message: attracts_description を rabbits_description に rename

File: urdf/mobile_base.xacro (robot description, xacro)
@@ -6,5 +6,5 @@
         <origin xyz="0 0 0" rpy="0 0 0" />
         <geometry>
-          <mesh filename="package://attracts_description/meshes/mobile_base.dae" scale="0.01 0.01 0.01"/>
+          <mesh filename="package://rabbits_description/meshes/mobile_base.dae" scale="0.01 0.01 0.01"/>
         </geometry>
       </visual>

File: urdf/proto1.xacro (robot description, xacro)
@@ -1,8 +1,8 @@
 <?xml version="1.0"?>
 <robot name="proto1" xmlns:xacro="http://ros.org/wiki/xacro">
-  <xacro:include filename="$(find attracts_description)/urdf/mobile_base.xacro" />
-  <xacro:include filename="$(find attracts_description)/urdf/wheel.xacro" />
-  <xacro:include filename="$(find attracts_description)/urdf/turret_base.xacro" />
-  <xacro:include filename="$(find attracts_description)/urdf/turret_unit.xacro" />
+  <xacro:include filename="$(find rabbits_description)/urdf/mobile_base.xacro" />
+  <xacro:include filename="$(find rabbits_description)/urdf/wheel.xacro" />
+  <xacro:include filename="$(find rabbits_description)/urdf/turret_base.xacro" />
+  <xacro:include filename="$(find rabbits_description)/urdf/turret_unit.xacro" />
   <xacro:mobile_base />
   <xacro:wheel prefix="right" suffix="front" />

File: urdf/turret_base.xacro (robot description, xacro)
@@ -6,5 +6,5 @@
         <origin xyz="0 0 0" rpy="0 0 0" />
         <geometry>
-          <mesh filename="package://attracts_description/meshes/turret_base.dae" scale="0.01 0.01 0.01"/>
+          <mesh filename="package://rabbits_description/meshes/turret_base.dae" scale="0.01 0.01 0.01"/>
         </geometry>
       </visual>

File: urdf/turret_unit.xacro (robot description, xacro)
@@ -6,5 +6,5 @@
         <origin xyz="0 0 0" rpy="0 0 0" />
         <geometry>
-          <mesh filename="package://attracts_description/meshes/turret_unit.dae" scale="0.01 0.01 0.01"/>
+          <mesh filename="package://rabbits_description/meshes/turret_unit.dae" scale="0.01 0.01 0.01"/>
         </geometry>
       </visual>

File: urdf/wheel.xacro (robot description, xacro)
@@ -6,5 +6,5 @@
         <origin xyz="0 0 0" rpy="0 0 0" />
         <geometry>
-          <mesh filename="package://attracts_description/meshes/wheel.dae" scale="0.01 0.01 0.01" />
+          <mesh filename="package://rabbits_description/meshes/wheel.dae" scale="0.01 0.01 0.01" />
         </geometry>
       </visual>
