Commit message: gamma の URDF を追加（寸法は仮）

File: urdf/proto1/mobile_base.xacro (robot description, xacro)
@@ -1,10 +1,10 @@
 <?xml version="1.0"?>
 <robot xmlns:xacro="http://ros.org/wiki/xacro">
-  <xacro:macro name="turret_unit">
-    <link name="pitch_link">
+  <xacro:macro name="mobile_base">
+    <link name="base_link">
       <visual>
         <origin xyz="0 0 0" rpy="0 0 0" />
         <geometry>
-          <mesh filename="package://rabbits_description/meshes/turret_unit.dae" scale="0.01 0.01 0.01"/>
+          <mesh filename="package://rabbits_description/meshes/proto1/mobile_base.dae" scale="0.01 0.01 0.01"/>
         </geometry>
       </visual>

File: urdf/proto1/proto1.xacro (robot description, xacro)
@@ -1,8 +1,8 @@
 <?xml version="1.0"?>
 <robot name="proto1" xmlns:xacro="http://ros.org/wiki/xacro">
-  <xacro:include filename="$(find rabbits_description)/urdf/mobile_base.xacro" />
-  <xacro:include filename="$(find rabbits_description)/urdf/wheel.xacro" />
-  <xacro:include filename="$(find rabbits_description)/urdf/turret_base.xacro" />
-  <xacro:include filename="$(find rabbits_description)/urdf/turret_unit.xacro" />
+  <xacro:include filename="$(find rabbits_description)/urdf/proto1/mobile_base.xacro" />
+  <xacro:include filename="$(find rabbits_description)/urdf/proto1/wheel.xacro" />
+  <xacro:include filename="$(find rabbits_description)/urdf/proto1/turret_base.xacro" />
+  <xacro:include filename="$(find rabbits_description)/urdf/proto1/turret_unit.xacro" />
   <xacro:mobile_base />
   <xacro:wheel prefix="right" suffix="front" />

File: urdf/proto1/turret_base.xacro (robot description, xacro)
@@ -1,14 +1,14 @@
 <?xml version="1.0"?>
 <robot xmlns:xacro="http://ros.org/wiki/xacro">
-  <xacro:macro name="wheel" params="prefix suffix">
-    <link name="${prefix}_${suffix}_wheel">
+  <xacro:macro name="turret_base">
+    <link name="yaw_link">
       <visual>
         <origin xyz="0 0 0" rpy="0 0 0" />
         <geometry>
-          <mesh filename="package://rabbits_description/meshes/wheel.dae" scale="0.01 0.01 0.01" />
+          <mesh filename="package://rabbits_description/meshes/proto1/turret_base.dae" scale="0.01 0.01 0.01"/>
         </geometry>
       </visual>
       <!-- <collision>
-        <origin xyz="0 0 0" rpy="${pi/2} 0 0" />
+        <origin xyz="0 0 0" rpy="0 0 0" />
       </collision> -->
       <inertial>

File: urdf/proto1/turret_unit.xacro (robot description, xacro)
@@ -1,10 +1,10 @@
 <?xml version="1.0"?>
 <robot xmlns:xacro="http://ros.org/wiki/xacro">
-  <xacro:macro name="turret_base">
-    <link name="yaw_link">
+  <xacro:macro name="turret_unit">
+    <link name="pitch_link">
       <visual>
         <origin xyz="0 0 0" rpy="0 0 0" />
         <geometry>
-          <mesh filename="package://rabbits_description/meshes/turret_base.dae" scale="0.01 0.01 0.01"/>
+          <mesh filename="package://rabbits_description/meshes/proto1/turret_unit.dae" scale="0.01 0.01 0.01"/>
         </geometry>
       </visual>

File: urdf/proto1/wheel.xacro (robot description, xacro)
@@ -1,14 +1,14 @@
 <?xml version="1.0"?>
 <robot xmlns:xacro="http://ros.org/wiki/xacro">
-  <xacro:macro name="mobile_base">
-    <link name="base_link">
+  <xacro:macro name="wheel" params="prefix suffix">
+    <link name="${prefix}_${suffix}_wheel">
       <visual>
         <origin xyz="0 0 0" rpy="0 0 0" />
         <geometry>
-          <mesh filename="package://rabbits_description/meshes/mobile_base.dae" scale="0.01 0.01 0.01"/>
+          <mesh filename="package://rabbits_description/meshes/proto1/wheel.dae" scale="0.01 0.01 0.01" />
         </geometry>
       </visual>
       <!-- <collision>
-        <origin xyz="0 0 0" rpy="0 0 0" />
+        <origin xyz="0 0 0" rpy="${pi/2} 0 0" />
       </collision> -->
       <inertial>
