Commit message: gamma の URDF に imu_link を追加

File: urdf/gamma/gamma.xacro (robot description, xacro)
@@ -26,4 +26,5 @@
   <xacro:property name="neck_pitch_offset" value="0.05" />
   <xacro:property name="neck_camera_offset" value="0.04" />
+  <xacro:property name="neck_imu_offset" value="0.03" />  <!-- カメラの後ろ。基板の位置が決まったら更新 -->
   <xacro:gamma_body size_xy="${body_size_xy}" height="${body_height}" />
   <!-- 脚 + 車輪。方位角は FR −45°, FL 45°, BR −135°, BL 135°（x 前、y 左） -->
@@ -42,4 +43,5 @@
   <!-- 首 -->
   <xacro:gamma_neck mount_z="${body_height / 2}" yaw_height="${neck_yaw_height}"
-                    pitch_offset="${neck_pitch_offset}" camera_offset="${neck_camera_offset}" />
+                    pitch_offset="${neck_pitch_offset}" camera_offset="${neck_camera_offset}"
+                    imu_offset="${neck_imu_offset}" />
 </robot>

File: urdf/gamma/neck.xacro (robot description, xacro)
@@ -2,10 +2,12 @@
 <!--
   gamma の首 3 軸（寸法は仮。CAD 確認後に差し替え）。
-  yaw_joint（z、continuous）→ pitch_joint（y、revolute）→ roll_joint（x、revolute）→ camera_link（固定。IMU とカメラ）。
+  yaw_joint（z、continuous）→ pitch_joint（y、revolute）→ roll_joint（x、revolute）→ camera_link（固定。カメラ）→ imu_link（固定）。
+  imu_link の向きは camera_link と同じ（回転なし）。軸の入れ替えはファームが BNO055 のレジスタで済ませ、imu/data を
+  カメラ座標系で出すので、TF で二重に回さない。位置は仮（カメラの後ろ imu_offset）。
   pitch / roll は論理関節（ファームが差動リンクの 2 モータ角から求めた値）。ロール軸を後回しにする間は 0 が来る。
   符号は REP-103: yaw 左が正、pitch 前が下がると正、roll 右が下がると正。
 -->
 <robot xmlns:xacro="http://ros.org/wiki/xacro">
-  <xacro:macro name="gamma_neck" params="mount_z yaw_height pitch_offset camera_offset">
+  <xacro:macro name="gamma_neck" params="mount_z yaw_height pitch_offset camera_offset imu_offset">
     <joint name="yaw_joint" type="continuous">
       <parent link="base_link" />
@@ -69,4 +71,19 @@
       </visual>
     </link>
+    <!-- IMU（BNO055、gamma_turret 基板上）。bridge の imu/data の frame_id -->
+    <joint name="imu_joint" type="fixed">
+      <parent link="camera_link" />
+      <child link="imu_link" />
+      <origin xyz="${-imu_offset} 0 0" rpy="0 0 0" />
+    </joint>
+    <link name="imu_link">
+      <visual>
+        <origin xyz="0 0 0" rpy="0 0 0" />
+        <geometry>
+          <box size="0.01 0.015 0.003" />
+        </geometry>
+        <material name="rabbits_blue" />
+      </visual>
+    </link>
   </xacro:macro>
 </robot>
