Commit message: 胴体に正面の目印を付ける

File: urdf/gamma/body.xacro (robot description, xacro)
@@ -11,4 +11,12 @@
         <material name="rabbits_grey" />
       </visual>
+      <!-- 正面（+x）の目印。カメラが yaw 0 で向く側 -->
+      <visual>
+        <origin xyz="${size_xy / 2 - 0.01} 0 ${height / 2 + 0.005}" rpy="0 0 0" />
+        <geometry>
+          <box size="0.02 ${size_xy * 0.6} 0.01" />
+        </geometry>
+        <material name="rabbits_orange" />
+      </visual>
     </link>
   </xacro:macro>

Commit message: gamma の脚を 4 節リンクの実寸にし、派生関節を出すミキサーを追加

File: urdf/gamma/body.xacro (robot description, xacro)
@@ -1,9 +1,9 @@
 <?xml version="1.0"?>
-<!-- gamma の胴体（寸法は仮。CAD 確認後に差し替え） -->
+<!-- gamma の胴体（寸法は仮。CAD 確認後に差し替え）。base 原点は脚モータ軸の面なので箱の中心は center_z -->
 <robot xmlns:xacro="http://ros.org/wiki/xacro">
-  <xacro:macro name="gamma_body" params="size_xy height">
+  <xacro:macro name="gamma_body" params="size_xy height center_z">
     <link name="base_link">
       <visual>
-        <origin xyz="0 0 0" rpy="0 0 0" />
+        <origin xyz="0 0 ${center_z}" rpy="0 0 0" />
         <geometry>
           <box size="${size_xy} ${size_xy} ${height}" />
@@ -13,5 +13,5 @@
       <!-- 正面（+x）の目印。カメラが yaw 0 で向く側 -->
       <visual>
-        <origin xyz="${size_xy / 2 - 0.01} 0 ${height / 2 + 0.005}" rpy="0 0 0" />
+        <origin xyz="${size_xy / 2 - 0.01} 0 ${center_z + height / 2 + 0.005}" rpy="0 0 0" />
         <geometry>
           <box size="0.02 ${size_xy * 0.6} 0.01" />

File: urdf/gamma/gamma.xacro (robot description, xacro)
@@ -1,5 +1,7 @@
 <?xml version="1.0"?>
 <!--
-  gamma（2026 年機）の URDF。寸法は仮（箱と円筒）。CAD 確認後にメッシュと寸法を差し替える。
+  gamma（2026 年機）の URDF。脚は 4 節リンクの実寸（config/gamma_linkage.yaml）、首と胴体は仮（箱と円筒）。
+  メッシュは README「gamma のメッシュの座標系」の約束で書き出したら差し替える。
+  base 原点 = 4 本の脚モータ軸を含む水平面と首 Yaw 軸の交点。x 前、y 左、z 上。
   軸の向きは設計書（rabbits_sim docs/superpowers/specs/2026-10-24-gamma-sim-design.md 5 章）の規約で確定:
     車輪は車輪リンクの z 軸が回転軸で z 正が機体の外側、脚は角度 0 が最下点で増えると車体が上がる。
@@ -8,5 +10,5 @@
     right_front_wheel_joint, left_front_wheel_joint, right_back_wheel_joint, left_back_wheel_joint,
     right_front_leg_joint, left_front_leg_joint, right_back_leg_joint, left_back_leg_joint
-  （*_knuckle_joint は mimic で、joint_states には載せない）
+  派生関節（*_bar_joint, *_coupler_joint）は linkage_state_publisher が足し、*_bar_lower_joint / *_holder_joint は mimic。
 -->
 <robot name="gamma" xmlns:xacro="http://ros.org/wiki/xacro">
@@ -15,33 +17,22 @@
   <xacro:include filename="$(find rabbits_description)/urdf/gamma/leg.xacro" />
   <xacro:include filename="$(find rabbits_description)/urdf/gamma/neck.xacro" />
-  <!-- 仮の寸法 [m] -->
-  <xacro:property name="body_size_xy" value="0.28" />
-  <xacro:property name="body_height" value="0.10" />
-  <xacro:property name="leg_radius" value="0.14" />        <!-- 脚の取り付け半径（gamma_turret_fw の BODY_D / 2） -->
-  <xacro:property name="leg_arm_length" value="0.10" />
-  <xacro:property name="leg_arm_radius" value="0.012" />
-  <xacro:property name="wheel_radius" value="0.03" />      <!-- WHEEL_D / 2 -->
-  <xacro:property name="wheel_width" value="0.02" />
-  <xacro:property name="neck_yaw_height" value="0.06" />
-  <xacro:property name="neck_pitch_offset" value="0.05" />
+  <!-- 寸法 [m / rad]。gamma_turret_fw の robot.hpp と対で更新する -->
+  <xacro:property name="cfg" value="${xacro.load_yaml('$(find rabbits_description)/config/gamma_linkage.yaml')}" />
+  <xacro:property name="L" value="${cfg['/**']['ros__parameters']['linkage']}" />
+  <!-- 仮の寸法 [m]（胴体の箱と首） -->
+  <xacro:property name="body_size_xy" value="0.24" />
+  <xacro:property name="body_height" value="0.08" />
+  <xacro:property name="body_center_z" value="-0.02" />   <!-- 脚モータ軸の面を跨ぐ -->
   <xacro:property name="neck_camera_offset" value="0.04" />
   <xacro:property name="neck_imu_offset" value="0.03" />  <!-- カメラの後ろ。基板の位置が決まったら更新 -->
-  <xacro:gamma_body size_xy="${body_size_xy}" height="${body_height}" />
+  <xacro:gamma_body size_xy="${body_size_xy}" height="${body_height}" center_z="${body_center_z}" />
   <!-- 脚 + 車輪。方位角は FR −45°, FL 45°, BR −135°, BL 135°（x 前、y 左） -->
-  <xacro:gamma_leg prefix="right_front" azimuth="${-pi / 4}" radius="${leg_radius}" mount_z="${-body_height / 2}"
-                   arm_length="${leg_arm_length}" arm_radius="${leg_arm_radius}"
-                   wheel_radius="${wheel_radius}" wheel_width="${wheel_width}" />
-  <xacro:gamma_leg prefix="left_front" azimuth="${pi / 4}" radius="${leg_radius}" mount_z="${-body_height / 2}"
-                   arm_length="${leg_arm_length}" arm_radius="${leg_arm_radius}"
-                   wheel_radius="${wheel_radius}" wheel_width="${wheel_width}" />
-  <xacro:gamma_leg prefix="right_back" azimuth="${-3 * pi / 4}" radius="${leg_radius}" mount_z="${-body_height / 2}"
-                   arm_length="${leg_arm_length}" arm_radius="${leg_arm_radius}"
-                   wheel_radius="${wheel_radius}" wheel_width="${wheel_width}" />
-  <xacro:gamma_leg prefix="left_back" azimuth="${3 * pi / 4}" radius="${leg_radius}" mount_z="${-body_height / 2}"
-                   arm_length="${leg_arm_length}" arm_radius="${leg_arm_radius}"
-                   wheel_radius="${wheel_radius}" wheel_width="${wheel_width}" />
-  <!-- 首 -->
-  <xacro:gamma_neck mount_z="${body_height / 2}" yaw_height="${neck_yaw_height}"
-                    pitch_offset="${neck_pitch_offset}" camera_offset="${neck_camera_offset}"
+  <xacro:gamma_leg prefix="right_front" azimuth="${-pi / 4}" L="${L}" />
+  <xacro:gamma_leg prefix="left_front" azimuth="${pi / 4}" L="${L}" />
+  <xacro:gamma_leg prefix="right_back" azimuth="${-3 * pi / 4}" L="${L}" />
+  <xacro:gamma_leg prefix="left_back" azimuth="${3 * pi / 4}" L="${L}" />
+  <!-- 首。Yaw 原点は実寸、Pitch / Roll は同じ点（仮） -->
+  <xacro:gamma_neck mount_z="${L['yaw_origin_z']}" yaw_height="${L['neck_pitch_z']}"
+                    pitch_offset="0" camera_offset="${neck_camera_offset}"
                     imu_offset="${neck_imu_offset}" />
 </robot>

File: urdf/gamma/leg.xacro (robot description, xacro)
@@ -1,56 +1,119 @@
 <?xml version="1.0"?>
 <!--
-  gamma の脚 1 本 + 車輪（寸法は仮。CAD 確認後に差し替え）。
-  関節の規約（設計書 rabbits_sim docs/superpowers/specs/2026-10-24-gamma-sim-design.md 5 章）:
-  - 脚の関節（<prefix>_leg_joint）: 原点は胴体の下面、方位角 azimuth の半径 radius の位置。
-    関節フレームの x = 半径方向外向き、y = 接線方向（z × x）、z = 上。回転軸は y。
-    角度 0 で腕は水平に外へ伸び、角度が増えると腕の先（車輪）が下がる = 車体が上がる。
-  - 車輪の関節（<prefix>_wheel_joint）: 車輪リンクの z 軸が回転軸で、z 正が機体の外側（半径方向）。
-  - ナックル（<prefix>_knuckle_joint）: 腕の先で −1 倍の mimic。平行リンクの「車輪の向きが胴体と平行のまま
-    上下する」振る舞いを表す。joint_states には載せない（robot_state_publisher が leg_joint から計算する）。
-  本物は平行リンクで、CAD で L / θ0 / r が分かったら 2 本目の腕も足して平行四辺形にする。
+  gamma の脚 1 本 + 車輪（4 節リンク、実寸。設計書 rabcl docs/superpowers/specs/2026-10-25-gamma-leg-linkage-design.md 7 章）。
+  寸法は config/gamma_linkage.yaml（引数 L）。見た目は箱と円筒（メッシュは後で差し替え）。
+  脚の面内 2 次元: 関節フレームは z 回りに方位角 azimuth だけ回し、x = 半径方向の外向き、z = 上。
+  回転軸はすべて +y（正の回転は x から −z へ = 下向き）。
+    base_link
+     ├─ <p>_leg_joint   （M、θ = joint_states の脚モータ角。0 = 車高が最も低い）→ crank_link
+     │    └─ <p>_coupler_joint（K、派生: −(ψ − α)）→ coupler_link（連結リンク。先端 J は閉じない = ループをここで切る）
+     ├─ <p>_bar_joint   （B1、派生: −φ）→ bar_link（上のバー）
+     │    └─ <p>_holder_joint（H1、mimic bar × −1）→ holder_link（車輪ホルダ。胴体と平行を保つ）
+     │         └─ <p>_wheel_joint（W、車輪の z = 半径方向の外向き）→ wheel
+     └─ <p>_bar_lower_joint（B2、mimic bar × 1）→ bar_lower_link（下のバー）
+  派生関節（bar、coupler）は linkage_state_publisher が rabcl::LegLinkage で計算して joint_states に足す。
+  クランクの向きは α = α0 − θ なので、クランクと連結リンクの visual は自分のフレームで +x から α0 上を向く。
 -->
 <robot xmlns:xacro="http://ros.org/wiki/xacro">
-  <xacro:macro name="gamma_leg" params="prefix azimuth radius mount_z arm_length arm_radius wheel_radius wheel_width">
-    <!-- 脚（腕）。関節フレームは z 回りに azimuth だけ回し、x を半径方向外向きにする -->
+  <xacro:macro name="gamma_leg" params="prefix azimuth L">
+    <xacro:property name="a0" value="${L['crank_angle_zero']}" />
+    <xacro:property name="Lc" value="${L['crank_length']}" />
+    <xacro:property name="Lr" value="${L['coupler_length']}" />
+    <xacro:property name="Lb" value="${L['bar_length']}" />
+    <xacro:property name="arm_r" value="0.006" />
+    <!-- クランク（脚モータの出力） -->
     <joint name="${prefix}_leg_joint" type="revolute">
       <parent link="base_link" />
-      <child link="${prefix}_leg_link" />
-      <origin xyz="${radius * cos(azimuth)} ${radius * sin(azimuth)} ${mount_z}" rpy="0 0 ${azimuth}" />
+      <child link="${prefix}_crank_link" />
+      <origin xyz="${L['leg_radius'] * cos(azimuth)} ${L['leg_radius'] * sin(azimuth)} 0" rpy="0 0 ${azimuth}" />
       <axis xyz="0 1 0" />
-      <limit lower="0" upper="1.6" effort="10" velocity="5" />
+      <limit lower="0" upper="${L['theta_max']}" effort="10" velocity="5" />
     </joint>
-    <link name="${prefix}_leg_link">
+    <link name="${prefix}_crank_link">
       <visual>
-        <origin xyz="${arm_length / 2} 0 0" rpy="0 ${pi / 2} 0" />
+        <origin xyz="${Lc / 2 * cos(a0)} 0 ${Lc / 2 * sin(a0)}" rpy="0 ${pi / 2 - a0} 0" />
         <geometry>
-          <cylinder radius="${arm_radius}" length="${arm_length}" />
+          <cylinder radius="${arm_r}" length="${Lc}" />
         </geometry>
         <material name="rabbits_blue" />
       </visual>
     </link>
-    <!-- ナックル: 腕の先。腕と逆に回って胴体と平行を保つ（平行リンクの従動側） -->
-    <joint name="${prefix}_knuckle_joint" type="revolute">
-      <parent link="${prefix}_leg_link" />
-      <child link="${prefix}_knuckle_link" />
-      <origin xyz="${arm_length} 0 0" rpy="0 0 0" />
+    <!-- 連結リンク（クランク先端 K にぶら下がる。先端 J はホルダに重なって見えるだけ） -->
+    <joint name="${prefix}_coupler_joint" type="revolute">
+      <parent link="${prefix}_crank_link" />
+      <child link="${prefix}_coupler_link" />
+      <origin xyz="${Lc * cos(a0)} 0 ${Lc * sin(a0)}" rpy="0 0 0" />
       <axis xyz="0 1 0" />
-      <limit lower="-1.6" upper="0" effort="10" velocity="5" />
-      <mimic joint="${prefix}_leg_joint" multiplier="-1" offset="0" />
+      <limit lower="${-pi}" upper="${pi}" effort="0" velocity="10" />
     </joint>
-    <link name="${prefix}_knuckle_link">
+    <link name="${prefix}_coupler_link">
       <visual>
-        <origin xyz="0 0 0" rpy="0 0 0" />
+        <origin xyz="${Lr / 2 * cos(a0)} 0 ${Lr / 2 * sin(a0)}" rpy="0 ${pi / 2 - a0} 0" />
         <geometry>
-          <sphere radius="${arm_radius * 1.5}" />
+          <cylinder radius="${arm_r}" length="${Lr}" />
         </geometry>
         <material name="rabbits_dark" />
       </visual>
     </link>
-    <!-- 車輪: z 軸が回転軸、z 正が機体の外側（ナックルの x = 半径方向外向き を z に向ける） -->
+    <!-- 上のバー（派生関節。バーのフレームでは +x 向き） -->
+    <joint name="${prefix}_bar_joint" type="revolute">
+      <parent link="base_link" />
+      <child link="${prefix}_bar_link" />
+      <origin xyz="${(L['leg_radius'] + L['bar_pivot'][0]) * cos(azimuth)} ${(L['leg_radius'] + L['bar_pivot'][0]) * sin(azimuth)} ${L['bar_pivot'][1]}"
+              rpy="0 0 ${azimuth}" />
+      <axis xyz="0 1 0" />
+      <limit lower="${-pi}" upper="${pi}" effort="0" velocity="10" />
+    </joint>
+    <link name="${prefix}_bar_link">
+      <visual>
+        <origin xyz="${Lb / 2} 0 0" rpy="0 ${pi / 2} 0" />
+        <geometry>
+          <cylinder radius="${arm_r}" length="${Lb}" />
+        </geometry>
+        <material name="rabbits_grey" />
+      </visual>
+    </link>
+    <!-- 下のバー（上のバーと同じ角度） -->
+    <joint name="${prefix}_bar_lower_joint" type="revolute">
+      <parent link="base_link" />
+      <child link="${prefix}_bar_lower_link" />
+      <origin xyz="${(L['leg_radius'] + L['bar_pivot_lower'][0]) * cos(azimuth)} ${(L['leg_radius'] + L['bar_pivot_lower'][0]) * sin(azimuth)} ${L['bar_pivot_lower'][1]}"
+              rpy="0 0 ${azimuth}" />
+      <axis xyz="0 1 0" />
+      <limit lower="${-pi}" upper="${pi}" effort="0" velocity="10" />
+      <mimic joint="${prefix}_bar_joint" multiplier="1" offset="0" />
+    </joint>
+    <link name="${prefix}_bar_lower_link">
+      <visual>
+        <origin xyz="${Lb / 2} 0 0" rpy="0 ${pi / 2} 0" />
+        <geometry>
+          <cylinder radius="${arm_r}" length="${Lb}" />
+        </geometry>
+        <material name="rabbits_grey" />
+      </visual>
+    </link>
+    <!-- ホルダ: 上のバーの先 H1。バーと逆に回って胴体と平行を保つ。J（上端ピン）と W（車輪中心）を含む -->
+    <joint name="${prefix}_holder_joint" type="revolute">
+      <parent link="${prefix}_bar_link" />
+      <child link="${prefix}_holder_link" />
+      <origin xyz="${Lb} 0 0" rpy="0 0 0" />
+      <axis xyz="0 1 0" />
+      <limit lower="${-pi}" upper="${pi}" effort="0" velocity="10" />
+      <mimic joint="${prefix}_bar_joint" multiplier="-1" offset="0" />
+    </joint>
+    <link name="${prefix}_holder_link">
+      <visual>
+        <origin xyz="${L['wheel'][0] / 2} 0 ${(L['coupler_pin'][1] + L['wheel'][1]) / 2}" rpy="0 0 0" />
+        <geometry>
+          <box size="${L['wheel'][0]} 0.02 ${L['coupler_pin'][1] - L['wheel'][1]}" />
+        </geometry>
+        <material name="rabbits_blue" />
+      </visual>
+    </link>
+    <!-- 車輪: z 軸が回転軸、z 正が機体の外側（ホルダの x = 半径方向外向き を z に向ける） -->
     <joint name="${prefix}_wheel_joint" type="continuous">
-      <parent link="${prefix}_knuckle_link" />
+      <parent link="${prefix}_holder_link" />
       <child link="${prefix}_wheel" />
-      <origin xyz="${wheel_width} 0 0" rpy="0 ${pi / 2} 0" />
+      <origin xyz="${L['wheel'][0]} 0 ${L['wheel'][1]}" rpy="0 ${pi / 2} 0" />
       <axis xyz="0 0 1" />
     </joint>
@@ -59,5 +122,5 @@
         <origin xyz="0 0 0" rpy="0 0 0" />
         <geometry>
-          <cylinder radius="${wheel_radius}" length="${wheel_width}" />
+          <cylinder radius="${L['wheel_radius']}" length="${L['wheel_width']}" />
         </geometry>
         <material name="rabbits_dark" />

File: urdf/gamma/neck.xacro (robot description, xacro)
@@ -34,7 +34,7 @@
     <link name="pitch_link">
       <visual>
-        <origin xyz="${pitch_offset / 2} 0 0" rpy="0 ${pi / 2} 0" />
+        <origin xyz="${pitch_offset / 2} 0 0" rpy="0 0 0" />
         <geometry>
-          <cylinder radius="0.02" length="${pitch_offset}" />
+          <sphere radius="0.02" />
         </geometry>
         <material name="rabbits_orange" />

Commit message: 胴体のメッシュを入れる

File: urdf/gamma/body.xacro (robot description, xacro)
@@ -1,22 +1,21 @@
 <?xml version="1.0"?>
-<!-- gamma の胴体（寸法は仮。CAD 確認後に差し替え）。base 原点は脚モータ軸の面なので箱の中心は center_z -->
+<!-- gamma の胴体（meshes/gamma/base.STL、mm、原点 = 脚モータ軸の水平面 × Yaw 軸、x 前・y 左・z 上）。
+     collision 用の箱は仮（center_z は脚モータ軸の面からの中心のずれ） -->
 <robot xmlns:xacro="http://ros.org/wiki/xacro">
   <xacro:macro name="gamma_body" params="size_xy height center_z">
     <link name="base_link">
       <visual>
+        <origin xyz="0 0 0" rpy="0 0 0" />
+        <geometry>
+          <mesh filename="package://rabbits_description/meshes/gamma/base.STL" scale="0.001 0.001 0.001" />
+        </geometry>
+        <material name="rabbits_grey" />
+      </visual>
+      <collision>
         <origin xyz="0 0 ${center_z}" rpy="0 0 0" />
         <geometry>
           <box size="${size_xy} ${size_xy} ${height}" />
         </geometry>
-        <material name="rabbits_grey" />
-      </visual>
-      <!-- 正面（+x）の目印。カメラが yaw 0 で向く側 -->
-      <visual>
-        <origin xyz="${size_xy / 2 - 0.01} 0 ${center_z + height / 2 + 0.005}" rpy="0 0 0" />
-        <geometry>
-          <box size="0.02 ${size_xy * 0.6} 0.01" />
-        </geometry>
-        <material name="rabbits_orange" />
-      </visual>
+      </collision>
     </link>
   </xacro:macro>
