Commit message: リンクを種類ごとに淡い色で分ける

File: urdf/common/materials.xacro (robot description, xacro)
@@ -14,3 +14,25 @@
     <color rgba="0.15 0.15 0.15 1.0" />
   </material>
+  <!-- 部品の種類ごとの色分け用。Fusion 360 のコンポーネント色循環のような淡い色 -->
+  <material name="rabbits_pale_blue">
+    <color rgba="0.60 0.76 0.93 1.0" />
+  </material>
+  <material name="rabbits_pale_green">
+    <color rgba="0.66 0.85 0.66 1.0" />
+  </material>
+  <material name="rabbits_pale_orange">
+    <color rgba="0.96 0.80 0.56 1.0" />
+  </material>
+  <material name="rabbits_pale_purple">
+    <color rgba="0.80 0.72 0.90 1.0" />
+  </material>
+  <material name="rabbits_pale_yellow">
+    <color rgba="0.95 0.90 0.62 1.0" />
+  </material>
+  <material name="rabbits_pale_grey">
+    <color rgba="0.78 0.78 0.80 1.0" />
+  </material>
+  <material name="rabbits_mid_grey">
+    <color rgba="0.35 0.35 0.38 1.0" />
+  </material>
 </robot>

File: urdf/gamma/body.xacro (robot description, xacro)
@@ -10,5 +10,5 @@
           <mesh filename="package://rabbits_description/meshes/gamma/base.STL" scale="0.001 0.001 0.001" />
         </geometry>
-        <material name="rabbits_grey" />
+        <material name="rabbits_pale_yellow" />
       </visual>
       <collision>

File: urdf/gamma/leg.xacro (robot description, xacro)
@@ -40,5 +40,5 @@
           <mesh filename="package://rabbits_description/meshes/gamma/crank.STL" scale="0.001 0.001 0.001" />
         </geometry>
-        <material name="rabbits_blue" />
+        <material name="rabbits_pale_blue" />
       </visual>
     </link>
@@ -57,5 +57,5 @@
           <mesh filename="package://rabbits_description/meshes/gamma/coupler.STL" scale="0.001 0.001 0.001" />
         </geometry>
-        <material name="rabbits_dark" />
+        <material name="rabbits_pale_orange" />
       </visual>
     </link>
@@ -75,5 +75,5 @@
           <mesh filename="package://rabbits_description/meshes/gamma/bar.STL" scale="0.001 0.001 0.001" />
         </geometry>
-        <material name="rabbits_grey" />
+        <material name="rabbits_pale_green" />
       </visual>
     </link>
@@ -94,5 +94,5 @@
           <mesh filename="package://rabbits_description/meshes/gamma/bar.STL" scale="0.001 0.001 0.001" />
         </geometry>
-        <material name="rabbits_grey" />
+        <material name="rabbits_pale_green" />
       </visual>
     </link>
@@ -113,5 +113,5 @@
           <mesh filename="package://rabbits_description/meshes/gamma/holder.STL" scale="0.001 0.001 0.001" />
         </geometry>
-        <material name="rabbits_blue" />
+        <material name="rabbits_pale_purple" />
       </visual>
     </link>
@@ -129,5 +129,5 @@
           <mesh filename="package://rabbits_description/meshes/gamma/wheel.STL" scale="0.001 0.001 0.001" />
         </geometry>
-        <material name="rabbits_dark" />
+        <material name="rabbits_mid_grey" />
       </visual>
     </link>
